Commit message: Drive the IGVC rover in Gazebo Fortress. Four wheel stand-ins and the Fortress diff-drive plugin so a keyboard cmd_vel yaws the chassis. Notes say this is not the official MARVIN model.

File: ros2/avl_description/urdf/tracked_rover.urdf.xacro (robot description, xacro)
@@ -62,10 +62,4 @@
       <material name="dark_grey"><color rgba="0.25 0.25 0.25 1"/></material>
     </visual>
-    <collision>
-      <origin xyz="0.3143 ${tread_y} ${xsens_height - 0.4763}" rpy="0 0 0"/>
-      <geometry>
-        <box size="${tread_length} ${tread_width} ${tread_height}"/>
-      </geometry>
-    </collision>
     <visual>
       <origin xyz="0.3143 ${-tread_y} ${xsens_height - 0.4763}" rpy="0 0 0"/>
@@ -75,10 +69,4 @@
       <material name="dark_grey"/>
     </visual>
-    <collision>
-      <origin xyz="0.3143 ${-tread_y} ${xsens_height - 0.4763}" rpy="0 0 0"/>
-      <geometry>
-        <box size="${tread_length} ${tread_width} ${tread_height}"/>
-      </geometry>
-    </collision>
     <!-- Source placeholder, not a measured mass. -->
     <inertial>
@@ -152,3 +140,52 @@
     <origin xyz="0.098 -0.286 ${xsens_height + 0.057}" rpy="0 0 -1.5708"/>
   </joint>
+  <!-- Track stand-ins. Separation is the surveyed tread centerline spacing. -->
+  <xacro:property name="wheel_radius" value="${tread_height / 2}"/>
+  <xacro:property name="wheel_separation" value="${tread_y * 2}"/>
+  <xacro:macro name="drive_wheel" params="prefix x y">
+    <link name="${prefix}_wheel">
+      <visual>
+        <origin xyz="0 0 0" rpy="${pi/2} 0 0"/>
+        <geometry>
+          <cylinder radius="${wheel_radius}" length="${tread_width}"/>
+        </geometry>
+        <material name="dark_grey"/>
+      </visual>
+      <collision>
+        <origin xyz="0 0 0" rpy="${pi/2} 0 0"/>
+        <geometry>
+          <cylinder radius="${wheel_radius}" length="${tread_width}"/>
+        </geometry>
+      </collision>
+      <inertial>
+        <mass value="2.0"/>
+        <inertia ixx="0.01" ixy="0" ixz="0" iyy="0.01" iyz="0" izz="0.01"/>
+      </inertial>
+    </link>
+    <joint name="${prefix}_wheel_joint" type="continuous">
+      <parent link="base_link"/>
+      <child link="${prefix}_wheel"/>
+      <origin xyz="${x} ${y} ${wheel_radius}" rpy="0 0 0"/>
+      <axis xyz="0 1 0"/>
+    </joint>
+  </xacro:macro>
+  <!-- Four contacts so the chassis cannot pitch onto its nose. -->
+  <xacro:drive_wheel prefix="left_rear" x="-0.05" y="${tread_y}"/>
+  <xacro:drive_wheel prefix="left_front" x="0.55" y="${tread_y}"/>
+  <xacro:drive_wheel prefix="right_rear" x="-0.05" y="${-tread_y}"/>
+  <xacro:drive_wheel prefix="right_front" x="0.55" y="${-tread_y}"/>
+  <gazebo>
+    <plugin filename="ignition-gazebo-diff-drive-system" name="ignition::gazebo::systems::DiffDrive">
+      <left_joint>left_rear_wheel_joint</left_joint>
+      <left_joint>left_front_wheel_joint</left_joint>
+      <right_joint>right_rear_wheel_joint</right_joint>
+      <right_joint>right_front_wheel_joint</right_joint>
+      <wheel_separation>${wheel_separation}</wheel_separation>
+      <wheel_radius>${wheel_radius}</wheel_radius>
+      <max_linear_velocity>1.0</max_linear_velocity>
+      <min_linear_velocity>-1.0</min_linear_velocity>
+      <max_angular_velocity>1.0</max_angular_velocity>
+      <min_angular_velocity>-1.0</min_angular_velocity>
+    </plugin>
+  </gazebo>
 </robot>

Commit message: fix sim frame names to match MARVIN contract

File: ros2/avl_description/urdf/tracked_rover.urdf.xacro (robot description, xacro)
@@ -2,13 +2,9 @@
 <!--
   Tracked rover for AVL Autonomy Sim.
-  Chassis and sensor mounts copied from Paarseus/IGVC_ROS2
+  Chassis geometry came from Paarseus/IGVC_ROS2
   src/avros_bringup/urdf/avros.urdf.xacro (Parsa Ghasemi, MIT).
-  That file credits a 2026-05-06 resurvey in cpp_avl_igvc/igvc_description.
-  Changes here:
-  - ZED X links are boxes at the same mount poses. The original includes
-    $(find zed_wrapper), which is not installed in this workspace.
-  - No wheel joints. This file is the rigid body only. Diff-drive comes later.
-  - Mass 150 kg and several mounts are still marked TODO in the source.
-    Do not treat them as assets/measurements.md.
+  Sensor frame names follow assets/urdf/frames.md. Mount transforms stay at
+  0 0 0 until they are measured and recorded in assets/measurements.md.
+  ZED optical frames use the normal ROS optical-frame orientation.
 -->
 <robot xmlns:xacro="http://www.ros.org/wiki/xacro" name="tracked_rover">
@@ -81,5 +77,5 @@
     <origin xyz="0 0 0" rpy="0 0 0"/>
   </joint>
-  <!-- TODO measure: source says sketch 2026-04-25, chassis center. -->
+  <!-- TODO measure: replace the zero mount from assets/measurements.md. -->
   <link name="imu_link">
     <visual>
@@ -91,7 +87,7 @@
     <parent link="base_link"/>
     <child link="imu_link"/>
-    <origin xyz="0 0 ${xsens_height}" rpy="0 0 0"/>
-  </joint>
-  <!-- TODO measure: source sketch, 3.5 in forward and 6.25 in up from the Xsens. -->
+    <origin xyz="0 0 0" rpy="0 0 0"/>
+  </joint>
+  <!-- TODO measure: replace the zero mount from assets/measurements.md. -->
   <link name="velodyne">
     <visual>
@@ -103,8 +99,15 @@
     <parent link="base_link"/>
     <child link="velodyne"/>
-    <origin xyz="0.089 0.0 ${xsens_height + 0.159}" rpy="0 0 0"/>
-  </joint>
-  <!-- Camera boxes stand in for zed_wrapper's zed_macro. Mounts match the source. -->
-  <link name="zed_front_camera_link">
+    <origin xyz="0 0 0" rpy="0 0 0"/>
+  </joint>
+  <!-- TODO measure: replace the zero mount from assets/measurements.md. -->
+  <link name="gps_link"/>
+  <joint name="gps_joint" type="fixed">
+    <parent link="base_link"/>
+    <child link="gps_link"/>
+    <origin xyz="0 0 0" rpy="0 0 0"/>
+  </joint>
+  <!-- Camera boxes stand in for zed_wrapper's zed_macro. -->
+  <link name="zed_center_link">
     <visual>
       <geometry><box size="0.04 0.17 0.03"/></geometry>
@@ -112,11 +115,11 @@
     </visual>
   </link>
-  <joint name="zed_front_mount_joint" type="fixed">
-    <parent link="base_link"/>
-    <child link="zed_front_camera_link"/>
-    <!-- Resurvey 2026-05-06: 26.75 in forward, 4.25 in below IMU. Pitch 15 deg down. -->
-    <origin xyz="0.6795 0.0 ${xsens_height - 0.108}" rpy="0 ${radians(15)} 0"/>
-  </joint>
-  <link name="zed_left_camera_link">
+  <joint name="zed_center_joint" type="fixed">
+    <parent link="base_link"/>
+    <child link="zed_center_link"/>
+    <!-- TODO measure -->
+    <origin xyz="0 0 0" rpy="0 0 0"/>
+  </joint>
+  <link name="zed_left_link">
     <visual>
       <geometry><box size="0.04 0.17 0.03"/></geometry>
@@ -124,10 +127,11 @@
     </visual>
   </link>
-  <joint name="zed_left_mount_joint" type="fixed">
-    <parent link="base_link"/>
-    <child link="zed_left_camera_link"/>
-    <origin xyz="0.098 0.286 ${xsens_height + 0.057}" rpy="0 0 1.5708"/>
-  </joint>
-  <link name="zed_right_camera_link">
+  <joint name="zed_left_joint" type="fixed">
+    <parent link="base_link"/>
+    <child link="zed_left_link"/>
+    <!-- TODO measure -->
+    <origin xyz="0 0 0" rpy="0 0 0"/>
+  </joint>
+  <link name="zed_right_link">
     <visual>
       <geometry><box size="0.04 0.17 0.03"/></geometry>
@@ -135,8 +139,28 @@
     </visual>
   </link>
-  <joint name="zed_right_mount_joint" type="fixed">
-    <parent link="base_link"/>
-    <child link="zed_right_camera_link"/>
-    <origin xyz="0.098 -0.286 ${xsens_height + 0.057}" rpy="0 0 -1.5708"/>
+  <joint name="zed_right_joint" type="fixed">
+    <parent link="base_link"/>
+    <child link="zed_right_link"/>
+    <!-- TODO measure -->
+    <origin xyz="0 0 0" rpy="0 0 0"/>
+  </joint>
+  <!-- Optical frames: x right, y down, z forward. -->
+  <link name="zed_left_optical_frame"/>
+  <joint name="zed_left_optical_joint" type="fixed">
+    <parent link="zed_left_link"/>
+    <child link="zed_left_optical_frame"/>
+    <origin xyz="0 0 0" rpy="-1.57079632679 0 -1.57079632679"/>
+  </joint>
+  <link name="zed_center_optical_frame"/>
+  <joint name="zed_center_optical_joint" type="fixed">
+    <parent link="zed_center_link"/>
+    <child link="zed_center_optical_frame"/>
+    <origin xyz="0 0 0" rpy="-1.57079632679 0 -1.57079632679"/>
+  </joint>
+  <link name="zed_right_optical_frame"/>
+  <joint name="zed_right_optical_joint" type="fixed">
+    <parent link="zed_right_link"/>
+    <child link="zed_right_optical_frame"/>
+    <origin xyz="0 0 0" rpy="-1.57079632679 0 -1.57079632679"/>
   </joint>
   <!-- Track stand-ins. Separation is the surveyed tread centerline spacing. -->

Commit message: Use the IGVC topic names and the Hosei course as the default sim world. The rover spawns on that course, and the topic map follows the IGVC stack instead of the old seed names.

File: ros2/avl_description/urdf/tracked_rover.urdf.xacro (robot description, xacro)
@@ -4,6 +4,7 @@
   Chassis geometry came from Paarseus/IGVC_ROS2
   src/avros_bringup/urdf/avros.urdf.xacro (Parsa Ghasemi, MIT).
-  Sensor frame names follow assets/urdf/frames.md. Mount transforms stay at
-  0 0 0 until they are measured and recorded in assets/measurements.md.
+  Sensor frame names follow assets/urdf/frames.md.
+  Mount numbers below are IGVC stand-ins (avros.urdf.xacro / avros_cam_sim),
+  except gps_link, which is still 0 0 0. Mass is 49 kg.
   ZED optical frames use the normal ROS optical-frame orientation.
 -->
@@ -65,8 +66,9 @@
       <material name="dark_grey"/>
     </visual>
-    <!-- Source placeholder, not a measured mass. -->
+    <!-- Whole robot is 49 kg. Four wheels are 1 kg each, so this link is 45 kg.
+         Inertia is the IGVC placeholder scaled by 45/150, not a CAD inertia. -->
     <inertial>
-      <mass value="150.0"/>
-      <inertia ixx="10.0" ixy="0" ixz="0" iyy="20.0" iyz="0" izz="25.0"/>
+      <mass value="45.0"/>
+      <inertia ixx="3.0" ixy="0" ixz="0" iyy="6.0" iyz="0" izz="7.5"/>
     </inertial>
   </link>
@@ -77,5 +79,5 @@
     <origin xyz="0 0 0" rpy="0 0 0"/>
   </joint>
-  <!-- TODO measure: replace the zero mount from assets/measurements.md. -->
+  <!-- IGVC stand-in from avros_cam_sim / avros.urdf.xacro. Not a measurements.md value. -->
   <link name="imu_link">
     <visual>
@@ -87,7 +89,7 @@
     <parent link="base_link"/>
     <child link="imu_link"/>
-    <origin xyz="0 0 0" rpy="0 0 0"/>
-  </joint>
-  <!-- TODO measure: replace the zero mount from assets/measurements.md. -->
+    <origin xyz="0 0 ${xsens_height}" rpy="0 0 0"/>
+  </joint>
+  <!-- IGVC stand-in: 3.5 in forward and 6.25 in above the IMU. Not a measurements.md value. -->
   <link name="velodyne">
     <visual>
@@ -99,12 +101,18 @@
     <parent link="base_link"/>
     <child link="velodyne"/>
-    <origin xyz="0 0 0" rpy="0 0 0"/>
-  </joint>
-  <!-- TODO measure: replace the zero mount from assets/measurements.md. -->
-  <link name="gps_link"/>
+    <origin xyz="0.089 0 ${xsens_height + 0.159}" rpy="0 0 0"/>
+  </joint>
+  <!-- On the roof of the main chassis, in line with the front camera. Not a tape measurement.
+       Roof height is the main-box center plus half its height. -->
+  <link name="gps_link">
+    <visual>
+      <geometry><box size="0.08 0.08 0.02"/></geometry>
+      <material name="gps_green"><color rgba="0.1 0.6 0.2 1"/></material>
+    </visual>
+  </link>
   <joint name="gps_joint" type="fixed">
     <parent link="base_link"/>
     <child link="gps_link"/>
-    <origin xyz="0 0 0" rpy="0 0 0"/>
+    <origin xyz="0.6795 0 ${xsens_height - 0.2191 + main_height / 2 + 0.01}" rpy="0 0 0"/>
   </joint>
   <!-- Camera boxes stand in for zed_wrapper's zed_macro. -->
@@ -118,6 +126,6 @@
     <parent link="base_link"/>
     <child link="zed_center_link"/>
-    <!-- TODO measure -->
-    <origin xyz="0 0 0" rpy="0 0 0"/>
+    <!-- IGVC stand-in. avros_cam_sim calls this zed_front. 15 deg down. -->
+    <origin xyz="0.6795 0 ${xsens_height - 0.108}" rpy="0 ${radians(15)} 0"/>
   </joint>
   <link name="zed_left_link">
@@ -130,6 +138,6 @@
     <parent link="base_link"/>
     <child link="zed_left_link"/>
-    <!-- TODO measure -->
-    <origin xyz="0 0 0" rpy="0 0 0"/>
+    <!-- IGVC stand-in. Faces left. -->
+    <origin xyz="0.098 0.286 ${xsens_height + 0.057}" rpy="0 0 1.5708"/>
   </joint>
   <link name="zed_right_link">
@@ -142,6 +150,6 @@
     <parent link="base_link"/>
     <child link="zed_right_link"/>
-    <!-- TODO measure -->
-    <origin xyz="0 0 0" rpy="0 0 0"/>
+    <!-- IGVC stand-in. Faces right. -->
+    <origin xyz="0.098 -0.286 ${xsens_height + 0.057}" rpy="0 0 -1.5708"/>
   </joint>
   <!-- Optical frames: x right, y down, z forward. -->
@@ -183,5 +191,5 @@
       </collision>
       <inertial>
-        <mass value="2.0"/>
+        <mass value="1.0"/>
         <inertia ixx="0.01" ixy="0" ixz="0" iyy="0.01" iyz="0" izz="0.01"/>
       </inertial>
